File: cell_sense.kicad_sch (KiCad schematic)
At the start: 10 parts

Commit message: Continued work on adding subcircuits for L99BM114
Parts:
- renumbered C12 to C4, R6 to R3, R7 to R4

Commit message: updated to use generics for passives
Parts:
- removed C1, C3: 10nF, PCM_JLCPCB:C_0402, symbol PCM_JLCPCB-Capacitors:0402,10nF
- removed R1, R3: 39R, symbol ct_lib:RTT20R039FTE
- removed R2, R4: 100Ω, PCM_JLCPCB:R_0402, symbol PCM_JLCPCB-Resistors:0402,100Ω
- added C11, C12: 10nF, symbol ct_lib:C
- added R4, R5: 39R, symbol ct_lib:R
- added R6, R7: 100R, symbol ct_lib:R
- renumbered C4 to C10, C2 to C9, FB1 to FB2, FB2 to FB3
Connections:
- net SENSE+: now also C11.2, C12.1, R6.2
- net SENSE-: now also C12.2, R7.2
- net SENSE_NEXT: now also C11.1
- net SOURCE: now also R5.2
- net SOURCE_NEXT: now also R4.2
- net at FB2.2: now also R6.1
- net at FB3.2: now also R7.1

Commit message: added BQ chip
Parts:
- removed C10, C9: 47nF, symbol ct_lib:CC0603KRX7R0BB473
- removed C11, C12: 10nF, symbol ct_lib:C
- removed FB2, FB3: 1kR 100MHz, symbol ct_lib:MPZ2012S102ATD25
- removed R4, R5: 39R, symbol ct_lib:R
- removed R6, R7: 100R, symbol ct_lib:R
