File: bms.kicad_sch (KiCad schematic)
At the start: 131 parts, among them J1 Conn_01x10, Q1 DMZ6012E, Q2 DMZ6012E, Q5 BSS123

Commit message: More sims, more buildout
Parts:
- removed C5: 470pF, PCM_JLCPCB:C_0402, symbol PCM_JLCPCB-Capacitors:0402,470pF
- removed J1: Conn_01x10, symbol Connector_Generic:Conn_01x10
- removed R?: 1m, symbol ct_lib:R
- added J1: Conn_01x08, symbol Connector_Generic:Conn_01x08
- added JP10, JP11, JP12, JP13, JP14, JP15, JP3, JP4, JP5, JP6, JP7, JP8, JP9: SolderJumper_2_Open, Jumper:SolderJumper-2_P1.3mm_Open_TrianglePad1.0x1.5mm, symbol Jumper:SolderJumper_2_Open
- R? (x17): value 330Ω -> 100Ω; symbol PCM_JLCPCB-Resistors:0402,330Ω -> PCM_JLCPCB-Resistors:0402,100Ω; LCSC C25104 -> C25076; Part 0402WGF3300TCE -> 0402WGF1000TCE; Resistance 330Ω -> 100Ω; Stock 1159127 -> 5907585; Temperature Coefficient ±100ppm/°C -> ±200ppm/°C
- R? (x16): value 82R -> 220Ω; symbol ct_lib:FRC0402J820_TS -> PCM_JLCPCB-Resistors:0402,220Ω; Attrition Qty (none) -> 10; Category (none) -> Resistors,Chip Resistor - Surface Mount; Class (none) -> Basic Component; LCSC (none) -> C25091; Manufacturer FOJAN -> UNI-ROYAL(Uniroyal Elec); Minimum Qty (none) -> 20; Operating Temperature Range (none) -> -55°C~+155°C; Overload Voltage (Max) (none) -> 50V; Part FRC0402J820 TS -> 0402WGF2200TCE; Power(Watts) (none) -> 62.5mW; Price (none) -> 0.004USD; Process (none) -> SMT; Resistance (none) -> 220Ω; Stock (none) -> 1127279; Temperature Coefficient (none) -> ±100ppm/°C; Tolerance (none) -> ±1%; Type (none) -> Thick Film Resistors
Connections:
- net CELLS_POSITIVE is gone; now on net TOP_CELL: D?.2
- net Cell0: now also J?.2 (Pin_2); no longer J?.1 (Pin_1)
- net Cell1: now also J?.3 (Pin_3); no longer J?.2 (Pin_2)
- net Cell10: now also J?.12 (Pin_12), JP7.1 (A), JP8.2 (B); no longer J?.11 (Pin_11)
- net Cell11: now also J?.13 (Pin_13), JP6.1 (A), JP7.2 (B); no longer J?.12 (Pin_12)
- net Cell12: now also J?.14 (Pin_14), JP5.1 (A), JP6.2 (B); no longer J?.13 (Pin_13)
- net Cell13: now also J?.15 (Pin_15), JP4.1 (A), JP5.2 (B); no longer J?.14 (Pin_14)
- net Cell14: now also J?.16 (Pin_16), JP3.1 (A), JP4.2 (B); no longer J?.15 (Pin_15)
- net Cell15: now also J?.17 (Pin_17), JP3.2 (B); no longer J?.16 (Pin_16)
- net Cell16: now also J?.18 (Pin_18); no longer J?.17 (Pin_17)
- net Cell2: now also J?.4 (Pin_4), JP15.1 (A); no longer J?.3 (Pin_3)
- net Cell3: now also J?.5 (Pin_5), JP14.1 (A), JP15.2 (B); no longer J?.4 (Pin_4)
- net Cell4: now also J?.6 (Pin_6), JP13.1 (A), JP14.2 (B); no longer J?.5 (Pin_5)
- net Cell5: now also J?.7 (Pin_7), JP12.1 (A), JP13.2 (B); no longer J?.6 (Pin_6)
- net Cell6: now also J?.8 (Pin_8), JP11.1 (A), JP12.2 (B); no longer J?.7 (Pin_7)
- net Cell7: now also J?.9 (Pin_9), JP10.1 (A), JP11.2 (B); no longer J?.8 (Pin_8)
- net Cell8: now also J?.10 (Pin_10), JP10.2 (B), JP9.1 (A); no longer J?.9 (Pin_9)
- net Cell9: now also J?.11 (Pin_11), JP8.1 (A), JP9.2 (B); no longer J?.10 (Pin_10)
- net GND: now also J?.1 (Pin_1), J1.2 (Pin_2), J1.4 (Pin_4), J1.6 (Pin_6), J1.8 (Pin_8)
- net TEMP1: now also J1.1 (Pin_1)
- net TEMP2: now also J1.3 (Pin_3)
- net TEMP3: now also J1.5 (Pin_5)
- net TEMP4: now also J1.7 (Pin_7)
- net VC0: now also R?.2; no longer R?.2
- net VC1: now also R?.2; no longer R?.2
- net VC10: now also R?.2; no longer R?.2
- net VC11: now also R?.2; no longer R?.2
- net VC12: now also R?.2; no longer R?.2
- net VC13: now also R?.2; no longer R?.2
- net VC14: now also R?.2; no longer R?.2
- net VC15: now also R?.2; no longer R?.2
- net VC2: now also R?.2; no longer R?.2
- net VC3: now also R?.2; no longer R?.2
- net VC4: now also R?.2; no longer R?.2
- net VC5: now also R?.2; no longer R?.2
- net VC6: now also R?.2; no longer R?.2
- net VC7: now also R?.2; no longer R?.2
- net VC8: now also R?.2; no longer R?.2
- net VC9: now also R?.2; no longer R?.2
- net at Q?.1 (B): now also R?.1; no longer R?.1 (x9)
- net FUSE_MEAS: now reaches Q5.1 (G), R11.1, R12.1
- net at R?.1: now also Q?.1 (B); no longer Q?.1 (B) (x5)
- net nWAKE: now reaches U?.22 (TS2/nWAKE)
- net PDSG_GATE_CTRL: now reaches U?.39 (PDSG)
- net TOP_CELL: now reaches J?.19 (Pin_19)
- net CELLS_NEGATIVE renamed CSENSE_N
- net OUTPUT_NEGATIVE renamed CSENSE_P
- net TEMP5 renamed ALERT
- net TEMP_CAL renamed TEMP_REF
- new net: Q?.1 (B), R?.1 (x2)
Other:
- note added: "*Required"
- note added: "Add tvs diodes to top cells"
- note added: "At a minimum, most populate calls at: VC0 -> VC1 VC1 -> VC2 VC15 -> VC16"
- note added: "Balancing / Cell Sense"
- note added: "Current Sense: -200 to 200 mV measurement -500 to 500 mV comparator"
- note added: "DO NOT USE TS2 FOR THERMISTOR Wakes up when pulled to ground (exits shutdown)"
- note added: "Fuse: Z if not permanent fault LOW if permanent fault Will set permanent fault if driven HIGH"
- note removed: "Balancing"
- note removed: "DO NOT USE TS2 Wakes up when pulled to ground (exits shutdown)"
- moved on the sheet: C1, C2, C3, C4, C6, C7, C8, C?, D3, D?, R13, R?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

Commit message: isolated comms
Parts:
- removed JP10, JP11, JP12, JP13, JP14, JP15, JP3, JP4, JP5, JP6, JP7, JP8, JP9: SolderJumper_2_Open, Jumper:SolderJumper-2_P1.3mm_Open_TrianglePad1.0x1.5mm, symbol Jumper:SolderJumper_2_Open
- added R38, R39, R40: 0Ω, PCM_JLCPCB:R_0402, symbol PCM_JLCPCB-Resistors:0402,0Ω
- added TP10, TP11, TP9: IO8, TestPoint:TestPoint_Pad_D1.0mm, symbol Connector:TestPoint
Connections:
- net LD: now also R38.1, R40.1, TP9.1; no longer D4.1, D?.1, Q2.3 (D)
- net PACK: now also R39.1, TP10.1; no longer D5.1, D?.1, Q1.3 (D)
- net nWAKE: now also TP11.1
- net AFE_BAT: now reaches C?.1, C?.1, C?.1, D3.2, R?.2, U?.47 (BAT)
- net AFE_BAT: now also R40.2
- net AFE_SDA renamed SDA
- net AFE_SDL renamed SDL
- new net: D5.1, D?.1, Q1.3 (D), R39.2
- new net: D4.1, D?.1, Q2.3 (D), R38.2
Other:
- note added: "Implement LDO"
- moved on the sheet: D4, D5, D?, Q1, Q2, R1, R2, R3, R8
