File: bms.kicad_sch (KiCad schematic)
At the start: 135 parts, among them J1 Conn_01x08, Q1 DMZ6012E, Q2 DMZ6012E, Q5 BSS123

Commit message: comms updates
Parts:
- added C12, C29: 1uF, PCM_JLCPCB:C_0402, symbol PCM_JLCPCB-Capacitors:0402,1uF
- added U8: XC6206P332MR, PCM_JLCPCB:SOT-23-3_L2.9-W1.6-P1.90-LS2.8-BR, symbol PCM_JLCPCB-Power:LDO, 3.3V, 0.2A
Connections:
- net GND: now also C12.2, C29.2, U8.1 (GND)
- new net 3V3: C29.1, U8.2 (VOUT)
- new net 5V0_SW: C12.1, U8.3 (VIN)
Other:
- note added: "3V3 Supply to MCU"
- moved on the sheet: D4, D5, D?, Q1, Q2, R1, R2, R3, R38, R39, R40, R8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

Commit message: adding diode or
Parts:
- added D20: BAT54C,215, PCM_JLCPCB:SOT-23-3_L2.9-W1.6-P1.90-LS2.8-BR, symbol PCM_JLCPCB-Diode-Packages:Schottky, BAT54C,215
Connections:
- net 5V0_SW: now also D20.2 (A); no longer C12.1, U8.3 (VIN)
- new net: C12.1, D20.3 (K), U8.3 (VIN)
Other:
- moved on the sheet: C12, C29, U8

Commit message: rolled back TO commit caa5444, didn't mean to roll THAT back
Parts:
- removed C? (x3): 470pF, PCM_JLCPCB:C_0402, symbol PCM_JLCPCB-Capacitors:0402,470pF
- removed C?: 100p, 100v, symbol ct_lib:C
- removed C?: 2.2u, 100v, symbol ct_lib:C
- added C30, C31: 1uF, PCM_JLCPCB:C_0402, symbol PCM_JLCPCB-Capacitors:0402,1uF
- added C32: 22nF, PCM_JLCPCB:C_0402, symbol PCM_JLCPCB-Capacitors:0402,22nF
- added C33: 1uF, PCM_JLCPCB:C_0805, symbol ct_lib:CC0805KKX7R0BB105
- added C34: 100pF, PCM_JLCPCB:C_0603, symbol ct_lib:CC0603JRNPO0BN101
- added C35: 2.2uF, PCM_JLCPCB:C_1206, symbol ct_lib:CC1206KKX7R0BB225
- added D21: BAT46W, PCM_JLCPCB:D_SOD-123, symbol PCM_JLCPCB-Diodes:Schottky,BAT46W
- added R67: 10MR, PCM_JLCPCB:R_0402, symbol ct_lib:RC0402JR-0710ML
- added R68: 100Ω, PCM_JLCPCB:R_0402, symbol PCM_JLCPCB-Resistors:0402,100Ω
- added R69, R70: 620R, PCM_JLCPCB:R_1206, symbol ct_lib:1206W4F6200T5E
- added U9: 2SC2383_C41375137, Package_TO_SOT_SMD:SOT-89-3, symbol JLCImport:2SC2383_C41375137
Connections:
- net AFE_BAT: now also C34.1, C35.1
- net GND: now also C30.2, C31.2, C32.2, C33.2, C34.2, C35.2, R67.2; no longer U?.36 (REGIN), U?.37 (BREG)
- net TOP_CELL: now also D21.2
- net at U?.24 (REG18): now also C31.1
- net REG1_5V0: now reaches D20.1 (A)
- net REG1_5V0: now also U?.35 (REG1), C30.1
- new net: R68.2, U9.1 (B)
- new net: C33.1, R69.2, R70.2, U9.2 (C)
- new net: D21.1, R69.1, R70.1
- new net BREG: R67.1, R68.1, U?.37 (BREG)
- new net REGIN: C32.1, U9.3 (E), U?.36 (REGIN)
- no-connect marks 1 -> 2
Other:
- note added: "Pop if power stage is not used"
- moved on the sheet: C12, C29, D20, U8

Commit message: Revert "added precharge circuit, filled in placeholder parts"
This reverts commit caa5444a50fe9d2ccb2e95970e40619801e9f697.
Parts:
- removed C30, C31: 1uF, PCM_JLCPCB:C_0402, symbol PCM_JLCPCB-Capacitors:0402,1uF
- removed C32: 22nF, PCM_JLCPCB:C_0402, symbol PCM_JLCPCB-Capacitors:0402,22nF
- removed C33: 1uF, PCM_JLCPCB:C_0805, symbol ct_lib:CC0805KKX7R0BB105
- removed C34: 100pF, PCM_JLCPCB:C_0603, symbol ct_lib:CC0603JRNPO0BN101
- removed C35: 2.2uF, PCM_JLCPCB:C_1206, symbol ct_lib:CC1206KKX7R0BB225
- removed D21: BAT46W, PCM_JLCPCB:D_SOD-123, symbol PCM_JLCPCB-Diodes:Schottky,BAT46W
- removed R67: 10MR, PCM_JLCPCB:R_0402, symbol ct_lib:RC0402JR-0710ML
- removed R68: 100Ω, PCM_JLCPCB:R_0402, symbol PCM_JLCPCB-Resistors:0402,100Ω
- removed R69, R70: 620R, PCM_JLCPCB:R_1206, symbol ct_lib:1206W4F6200T5E
- removed U9: 2SC2383_C41375137, Package_TO_SOT_SMD:SOT-89-3, symbol JLCImport:2SC2383_C41375137
- added C? (x3): 470pF, PCM_JLCPCB:C_0402, symbol PCM_JLCPCB-Capacitors:0402,470pF
- added C?: 100p, 100v, symbol ct_lib:C
- added C?: 2.2u, 100v, symbol ct_lib:C
Connections:
- net BREG is gone; now on net GND: U?.37 (BREG)
- net REGIN is gone; now on net GND: U?.36 (REGIN)
- net AFE_BAT: now also C?.1, C?.1
- net GND: now also C?.2, C?.2, C?.2, C?.2, C?.2
- net at U?.24 (REG18): now also C?.1
- net at U?.34 (REG2): now also C?.1
- net REG1_5V0: no longer names the net of D20.1 (A)
- net REG1_5V0: no longer U?.35 (REG1)
- new net: C?.1, U?.35 (REG1)
- no-connect marks 2 -> 1
Other:
- note removed: "Pop if power stage is not used"
- moved on the sheet: C12, C29, D20, U8
