File: bms.kicad_sch (KiCad schematic)
At the start: 146 parts, among them J1 Conn_01x08, Q1 DMZ6012E, Q2 DMZ6012E, Q5 BSS123, U8 XC6206P332MR, U9 2SC2383_C41375137

Commit message: prepping for split into 2 boards
Parts:
- removed C1, C2, C3, C4, C6, C7, C8: 470pF, PCM_JLCPCB:C_0402, symbol PCM_JLCPCB-Capacitors:0402,470pF
- removed J1: Conn_01x08, symbol Connector_Generic:Conn_01x08
- removed R13: 18kR, PCM_JLCPCB:R_0402, symbol ct_lib:RT0402BRD0718KL
- removed R38, R39: 0Ω, PCM_JLCPCB:R_0402, symbol PCM_JLCPCB-Resistors:0402,0Ω
- removed TH1, TH2: 10k, PCM_JLCPCB:R_0402, symbol ct_lib:B57232V5103F360
- added C36, C37, C38, C39, C40: 470pF, PCM_JLCPCB:C_0402, symbol PCM_JLCPCB-Capacitors:0402,470pF
- added J5: Conn_02x07_Odd_Even, symbol Connector_Generic:Conn_02x07_Odd_Even
- added J9: Conn_01x08, symbol Connector_Generic:Conn_01x08
- added JP6: SolderJumper_2_Open, Jumper:SolderJumper-2_P1.3mm_Open_RoundedPad1.0x1.5mm, symbol Jumper:SolderJumper_2_Open
- added R36: 18kR, PCM_JLCPCB:R_0402, symbol ct_lib:RT0402BRD0718KL
- R40: now fitted
Connections:
- net AFE_BAT: no longer R40.2
- net CHARGE_PUMP: now also J5.5 (Pin_5)
- net CHG_GATE_CTRL: now also J5.7 (Pin_7)
- net GND: now also C37.2, C38.2, C39.2, C40.2, J5.1 (Pin_1), J9.2 (Pin_2), J9.4 (Pin_4), J9.6 (Pin_6), J9.8 (Pin_8), R36.2
- net LD: now also D4.1, D?.1, Q2.3 (D); no longer R40.1
- net PACK: now also D5.1, D?.1, Q1.3 (D)
- net PDSG_GATE_CTRL: now also J5.11 (Pin_11)
- net TEMP_CHG: now also J5.4 (Pin_4); no longer U?.29 (CFETOFF)
- net TEMP_DSG: now also J5.2 (Pin_2); no longer U?.30 (DFETOFF)
- net TEMP_REF: now also C40.1, R36.1
- net TOP_CELL: now also J5.3 (Pin_3)
- net CSENSE_N renamed CURRENT_SENSE_N
- net CURRENT_SENSE_N: now also J5.14 (Pin_14), JP6.1 (A)
- net CSENSE_P renamed CURRENT_SENSE_P
- net CURRENT_SENSE_P: now also J5.12 (Pin_12), JP6.2 (B)
- net DSG_GATE_CTRL renamed DSG_GATE_CONTROL
- net DSG_GATE_CONTROL: now also J5.9 (Pin_9)
- net OUTPUT_POSITIVE renamed PACK/LD
- net PACK/LD: now also R40.2, J5.13 (Pin_13)
- net TEMP3 renamed DDSG
- net DDSG: now also J5.6 (Pin_6)
- net TEMP4 renamed DCHG
- net DCHG: now also J5.8 (Pin_8)
- new net FUSE: J5.10 (Pin_10)
- new net TEMP_CELLS_1: C36.1, J9.1 (Pin_1)
- new net TEMP_CELLS_2: C37.1, J9.3 (Pin_3)
- new net TEMP_CELLS_3: C38.1, J9.5 (Pin_5)
- new net TEMP_CELLS_4: C39.1, J9.7 (Pin_7)
- new net TEMP_CHG_FETS: U?.29 (CFETOFF)
- new net TEMP_DSG_FETS: U?.30 (DFETOFF)
Other:
- note added: "Thermistor Reference"
- note added: "To Power Stage"
- note removed: "Pop if power stage is not used"
- moved on the sheet: C12, C29, C32, C33, D20, D21, D4, D5, D?, J?, Q1, Q2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
