File: CAN.kicad_sch (KiCad schematic)
At the start: 42 parts, among them J4 Connector, USB-TYPE-C-16P, J6 Conn_01x04, U2 ISO1042BDWVR, U3 MIE1W0505BGLVH-3R-Z, U4 MP9485GN-Z, U5 HT7533, U6 ADUM3160, U7 LTV-217-B-G

Commit message: 10.0
Other:
- moved on the sheet: R53, U7

Commit message: comms updates
Parts:
- removed C12, C21, C22: 10uF, PCM_JLCPCB:C_0603, symbol PCM_JLCPCB-Capacitors:0603,10uF
- removed JP16: SolderJumper_2_Open, Jumper:SolderJumper-2_P1.3mm_Open_RoundedPad1.0x1.5mm, symbol Jumper:SolderJumper_2_Open
- removed R37: 120Ω, PCM_JLCPCB:R_1206, symbol PCM_JLCPCB-Resistors:1206,120Ω
- removed TP6: IO8, TestPoint:TestPoint_Pad_D1.0mm, symbol Connector:TestPoint
- removed U2: ISO1042BDWVR, ct_lib:ISO1042BDWVR, symbol ct_lib:ISO1042BDWVR
- removed U5: HT7533, PCM_JLCPCB:SOT-89-3_L4.5-W2.5-P1.50-LS4.2-BR, symbol PCM_JLCPCB-Power:LDO, 3.3V, 0.1A
- added C21, C22, C27, C28: 100uF, PCM_JLCPCB:C_1206, symbol PCM_JLCPCB-Capacitors:1206,100uF
- added C25, C26: 100nF, PCM_JLCPCB:C_0402, symbol PCM_JLCPCB-Capacitors:0402,100nF
- added D19: BAT20JFILM, PCM_JLCPCB:SOT-323-3_L2.0-W1.3-P1.30-LS2.3-BR, symbol JLCImport:BAT20JFILM
- added JP3: Jumper_2_Open, Jumper:SolderJumper-2_P1.3mm_Open_RoundedPad1.0x1.5mm, symbol Jumper:Jumper_2_Open
- added JP4: SolderJumper_2_Open, symbol Jumper:SolderJumper_2_Open
- added R37: 120Ω, PCM_JLCPCB:R_0402, symbol PCM_JLCPCB-Resistors:0402,120Ω
- added R54: 0Ω, PCM_JLCPCB:R_0402, symbol PCM_JLCPCB-Resistors:0402,0Ω
- added R55: 100kΩ, PCM_JLCPCB:R_0402, symbol PCM_JLCPCB-Resistors:0402,100kΩ
- added TP14, TP15, TP16, TP17, TP18, TP19: IO8, TestPoint:TestPoint_Pad_D1.0mm, symbol Connector:TestPoint
- added U2: TCAN334D, ct_lib:TCAN334D, symbol ct_lib:TCAN334D
- added U5: ISO7041FDBQ, Package_SO:SOIC-16W_7.5x10.3mm_P1.27mm, symbol ct_lib:ISO7041FDBQ
- R42: now not fitted
Connections:
- net nEN_ISO_PWR is gone; now on net EN_ISO_PWR: U4.6 (DIM), U4.7 (~{EN})
- net 5V0_ISO_SW: now also C21.1, C22.1, C27.1, C28.1, D19.1 (K), TP14.1, U2.3 (VCC1), U5.16 (VCC2); no longer C13.1, TP7.1, U3.5,6 (VOUT)
- net 5V0_SW: now also C25.1; no longer C23.2
- net CAN_RX: now also TP15.1, U5.6 (OUTD)
- net CAN_TX: now also TP16.1, U5.5 (INC)
- net GND: now also C23.2, C24.1, C25.2, C26.2
- net GNDISO: now also C13.2, U3.2 (GND2), U3.3,4 (GND2), C21.2, C22.2, C27.2, C28.2, R54.2, TP17.1, U2.2 (GND), U5.15 (GND2), U5.9 (GND2)
- net USB_nINT: now also R55.2
- net at J6.2 (Pin_2): now also D17.1 (K), R37.1, U2.7 (CANH); no longer D17.2 (K)
- net at R51.2, U6.14 (VDD2): now also C24.2; no longer C24.1
- net at R46.1, U6.16 (VBUS2): now also C26.1; no longer C24.2
- net USB_ISO_P: now reaches J4.A6 (D+), J4.B6 (D+), U6.10 (DD+)
- net USB_ISO_N: now reaches J4.A7 (D-), J4.B7 (D-), U6.11 (DD-)
- net EN_ISO_PWR: now reaches R42.2, U3.8 (EN)
- net at J6.3 (Pin_3): now also D17.2 (K), JP3.1 (A), U2.6 (CANL); no longer D17.1 (K)
- new net: C13.1, D19.2 (A), TP7.1, U3.5,6 (VOUT)
- new net: JP4.2 (B), R54.1, U2.5 (SHDN)
- new net: JP3.2 (B), R37.2
- new net: U2.4 (RXD), U5.11 (IND)
- new net: U2.1 (TXD), U5.12 (OUTC)
- new net: JP4.1 (A), U5.13 (OUTB)
- new net: U2.8 (STB), U5.14 (OUTA)
- new net: U5.2 (GND1), U5.8 (GND1)
- new net 3V3: R55.1
- new net CAN_SHUTDOWN: TP18.1, U5.4 (INB)
- new net CAN_SLEEP: TP19.1, U5.3 (INA)
- no-connect marks 2 -> 4
Other:
- note added: "5V Isolated Switched for CAN"
- note added: "Chip Quiescent: 5uA OFF 250uaA ON"
- note added: "Higher current 5V DC-DC supply for comms interfaces"
- note added: "On: HIGH Off: LOW"
- note removed: "3V3 Switched"
- note removed: "5V Isolated Switched"
- note removed: "Wow this is all just for isolated CAN... Why not just use a Bluetooth to CAN converter"
- moved on the sheet: C10, C13, C14, C15, C16, C17, C18, C19, C20, C5, D18, J4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

Commit message: adding diode or
Parts:
- added R66: 100kΩ, PCM_JLCPCB:R_0402, symbol PCM_JLCPCB-Resistors:0402,100kΩ
Connections:
- net EN_ISO_PWR: now also R66.1
- net GND: now also R66.2

Commit message: rolled back TO commit caa5444, didn't mean to roll THAT back
Connections:
- net GND: now also U5.2 (GND1), U5.8 (GND1); no longer C26.2
- net GNDISO: now also C26.2
Changed lines of the file:
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@@
 	)
 	(junction
-		(at 231.14 40.64)
-		(diameter 0)
-		(color 0 0 0 0)
-	)
-	(junction
 		(at 233.68 76.2)
 		(diameter 0)
@@
 	(wire
 		(pts
-			(xy 231.14 40.64) (xy 232.41 40.64)
-		)
-		(stroke
-			(width 0)
-			(type default)
-		)
-	)
-	(wire
-		(pts
 			(xy 231.14 68.58) (xy 228.6 68.58)
 		)
@@
 	(wire
 		(pts
+			(xy 231.14 134.62) (xy 233.68 134.62)
+		)
+		(stroke
+			(width 0)
+			(type default)
+		)
+	)
+	(wire
+		(pts
 			(xy 226.06 176.53) (xy 226.06 177.8)
 		)
@@
 	)
 	(symbol
+		(lib_id "power:Earth")
+		(at 261.62 177.8 0)
+		(unit 1)
+		(body_style 1)
+		(exclude_from_sim no)
+		(in_bom yes)
+		(on_board yes)
+		(in_pos_files yes)
+		(dnp no)
+		(fields_autoplaced yes)
+		(property "Reference" "#PWR051"
+			(at 261.62 184.15 0)
+			(hide yes)
+			(show_name no)
+			(do_not_autoplace no)
+			(effects
+				(font
+					(size 1.27 1.27)
+				)
+			)
+		)
+		(property "Value" "GNDISO"
+			(at 261.62 181.9331 0)
+			(show_name no)
+			(do_not_autoplace no)
+			(effects
+				(font
+					(size 1.27 1.27)
+				)
+			)
+		)
+		(property "Footprint" ""
+			(at 261.62 177.8 0)
+			(hide yes)
+			(show_name no)
+			(do_not_autoplace no)
+			(effects
+				(font
+					(size 1.27 1.27)
+				)
+			)
+		)
+		(property "Datasheet" ""
+			(at 261.62 177.8 0)
+			(hide yes)
+			(show_name no)
+			(do_not_autoplace no)
+			(effects
+				(font
+					(size 1.27 1.27)
+				)
+			)
+		)
+		(property "Description" "Power symbol creates a global label with name \"GNDISO\""
+			(at 261.62 177.8 0)
+			(hide yes)
+			(show_name no)
+			(do_not_autoplace no)
+			(effects
+				(font
+					(size 1.27 1.27)
+				)
+			)
+		)
+		(pin "1"
+		)
+		(instances
+			(project "battery-node"
+				(path "/0531bb65-44fe-462a-8fbf-92fb22c9abe0/a0e287d3-b915-410a-86a7-dfb59e4205a2"
+					(reference "#PWR051")
+					(unit 1)
+				)
+			)
+		)
+	)
+	(symbol
 		(lib_id "PCM_JLCPCB-Resistors:0402,0Ω")
 		(at 257.81 214.63 0)
@@
 	)
 	(symbol
-		(lib_id "power:GND")
-		(at 261.62 177.8 0)
-		(unit 1)
-		(body_style 1)
-		(exclude_from_sim no)
-		(in_bom yes)
-		(on_board yes)
-		(in_pos_files yes)
-		(dnp no)
-		(fields_autoplaced yes)
-		(property "Reference" "#PWR051"
-			(at 261.62 184.15 0)
-			(hide yes)
-			(show_name no)
-			(do_not_autoplace no)
-			(effects
-				(font
-					(size 1.27 1.27)
-				)
-			)
-		)
-		(property "Value" "GND"
-			(at 261.62 181.9331 0)
-			(show_name no)
-			(do_not_autoplace no)
-			(effects
-				(font
-					(size 1.27 1.27)
-				)
-			)
-		)
-		(property "Footprint" ""
-			(at 261.62 177.8 0)
-			(hide yes)
-			(show_name no)
-			(do_not_autoplace no)
-			(effects
-				(font
-					(size 1.27 1.27)
-				)
-			)
-		)
-		(property "Datasheet" ""
-			(at 261.62 177.8 0)
-			(hide yes)
-			(show_name no)
-			(do_not_autoplace no)
-			(effects
-				(font
-					(size 1.27 1.27)
-				)
-			)
-		)
-		(property "Description" "Power symbol creates a global label with name \"GND\" , ground"
-			(at 261.62 177.8 0)
-			(hide yes)
-			(show_name no)
-			(do_not_autoplace no)
-			(effects
-				(font
-					(size 1.27 1.27)
-				)
-			)
-		)
-		(pin "1"
-		)
-		(instances
-			(project "battery-node"
-				(path "/0531bb65-44fe-462a-8fbf-92fb22c9abe0/a0e287d3-b915-410a-86a7-dfb59e4205a2"
-					(reference "#PWR051")
-					(unit 1)
-				)
-			)
-		)
-	)
-	(symbol
 		(lib_id "power:+3V3")
 		(at 208.28 168.91 90)
@@
 					(unit 1)
 				)
+			)
+		)
+	)
+	(symbol
+		(lib_id "power:GND")
+		(at 231.14 134.62 0)
+		(unit 1)
+		(body_style 1)
+		(exclude_from_sim no)
+		(in_bom yes)
+		(on_board yes)
+		(in_pos_files yes)
+		(dnp no)
+		(fields_autoplaced yes)
+		(property "Reference" "#PWR061"
+			(at 231.14 140.97 0)
+			(hide yes)
+			(show_name no)
+			(do_not_autoplace no)
+			(effects
+				(font
+					(size 1.27 1.27)
+				)
+			)
+		)
+		(property "Value" "GND"
+			(at 231.14 138.7531 0)
+			(show_name no)
+			(do_not_autoplace no)
+			(effects
+				(font
+					(size 1.27 1.27)
+				)
+			)
+		)
+		(property "Footprint" ""
+			(at 231.14 134.62 0)
+			(hide yes)
+			(show_name no)
+			(do_not_autoplace no)
+			(effects
+				(font
+					(size 1.27 1.27)
+				)
+			)
+		)
+		(property "Datasheet" ""
+			(at 231.14 134.62 0)
+			(hide yes)
+			(show_name no)
+			(do_not_autoplace no)
+			(effects
+				(font
+					(size 1.27 1.27)
+				)
+			)
+		)
+		(property "Description" "Power symbol creates a global label with name \"GND\" , ground"
+			(at 231.14 134.62 0)
+			(hide yes)
+			(show_name no)
+			(do_not_autoplace no)
+			(effects
+				(font
+					(size 1.27 1.27)
+				)
+			)
+		)
+		(pin "1"
+		)
+		(instances
+			(project "battery-node"
+				(path "/0531bb65-44fe-462a-8fbf-92fb22c9abe0/a0e287d3-b915-410a-86a7-dfb59e4205a2"
+					(reference "#PWR061")
+					(unit 1)
+				)

Commit message: Revert "added precharge circuit, filled in placeholder parts"
This reverts commit caa5444a50fe9d2ccb2e95970e40619801e9f697.
Connections:
- net GND: now also C26.2; no longer U5.2 (GND1), U5.8 (GND1)
- net GNDISO: no longer C26.2
- new net: U5.2 (GND1), U5.8 (GND1)
Changed lines of the file:
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@@
 	)
 	(junction
+		(at 231.14 40.64)
+		(diameter 0)
+		(color 0 0 0 0)
+	)
+	(junction
 		(at 233.68 76.2)
 		(diameter 0)
@@
 	(wire
 		(pts
+			(xy 231.14 40.64) (xy 232.41 40.64)
+		)
+		(stroke
+			(width 0)
+			(type default)
+		)
+	)
+	(wire
+		(pts
 			(xy 231.14 68.58) (xy 228.6 68.58)
 		)
@@
 	(wire
 		(pts
-			(xy 231.14 134.62) (xy 233.68 134.62)
-		)
-		(stroke
-			(width 0)
-			(type default)
-		)
-	)
-	(wire
-		(pts
 			(xy 226.06 176.53) (xy 226.06 177.8)
 		)
@@
 	)
 	(symbol
-		(lib_id "power:Earth")
-		(at 261.62 177.8 0)
-		(unit 1)
-		(body_style 1)
-		(exclude_from_sim no)
-		(in_bom yes)
-		(on_board yes)
-		(in_pos_files yes)
-		(dnp no)
-		(fields_autoplaced yes)
-		(property "Reference" "#PWR051"
-			(at 261.62 184.15 0)
-			(hide yes)
-			(show_name no)
-			(do_not_autoplace no)
-			(effects
-				(font
-					(size 1.27 1.27)
-				)
-			)
-		)
-		(property "Value" "GNDISO"
-			(at 261.62 181.9331 0)
-			(show_name no)
-			(do_not_autoplace no)
-			(effects
-				(font
-					(size 1.27 1.27)
-				)
-			)
-		)
-		(property "Footprint" ""
-			(at 261.62 177.8 0)
-			(hide yes)
-			(show_name no)
-			(do_not_autoplace no)
-			(effects
-				(font
-					(size 1.27 1.27)
-				)
-			)
-		)
-		(property "Datasheet" ""
-			(at 261.62 177.8 0)
-			(hide yes)
-			(show_name no)
-			(do_not_autoplace no)
-			(effects
-				(font
-					(size 1.27 1.27)
-				)
-			)
-		)
-		(property "Description" "Power symbol creates a global label with name \"GNDISO\""
-			(at 261.62 177.8 0)
-			(hide yes)
-			(show_name no)
-			(do_not_autoplace no)
-			(effects
-				(font
-					(size 1.27 1.27)
-				)
-			)
-		)
-		(pin "1"
-		)
-		(instances
-			(project "battery-node"
-				(path "/0531bb65-44fe-462a-8fbf-92fb22c9abe0/a0e287d3-b915-410a-86a7-dfb59e4205a2"
-					(reference "#PWR051")
-					(unit 1)
-				)
-			)
-		)
-	)
-	(symbol
 		(lib_id "PCM_JLCPCB-Resistors:0402,0Ω")
 		(at 257.81 214.63 0)
@@
 	)
 	(symbol
+		(lib_id "power:GND")
+		(at 261.62 177.8 0)
+		(unit 1)
+		(body_style 1)
+		(exclude_from_sim no)
+		(in_bom yes)
+		(on_board yes)
+		(in_pos_files yes)
+		(dnp no)
+		(fields_autoplaced yes)
+		(property "Reference" "#PWR051"
+			(at 261.62 184.15 0)
+			(hide yes)
+			(show_name no)
+			(do_not_autoplace no)
+			(effects
+				(font
+					(size 1.27 1.27)
+				)
+			)
+		)
+		(property "Value" "GND"
+			(at 261.62 181.9331 0)
+			(show_name no)
+			(do_not_autoplace no)
+			(effects
+				(font
+					(size 1.27 1.27)
+				)
+			)
+		)
+		(property "Footprint" ""
+			(at 261.62 177.8 0)
+			(hide yes)
+			(show_name no)
+			(do_not_autoplace no)
+			(effects
+				(font
+					(size 1.27 1.27)
+				)
+			)
+		)
+		(property "Datasheet" ""
+			(at 261.62 177.8 0)
+			(hide yes)
+			(show_name no)
+			(do_not_autoplace no)
+			(effects
+				(font
+					(size 1.27 1.27)
+				)
+			)
+		)
+		(property "Description" "Power symbol creates a global label with name \"GND\" , ground"
+			(at 261.62 177.8 0)
+			(hide yes)
+			(show_name no)
+			(do_not_autoplace no)
+			(effects
+				(font
+					(size 1.27 1.27)
+				)
+			)
+		)
+		(pin "1"
+		)
+		(instances
+			(project "battery-node"
+				(path "/0531bb65-44fe-462a-8fbf-92fb22c9abe0/a0e287d3-b915-410a-86a7-dfb59e4205a2"
+					(reference "#PWR051")
+					(unit 1)
+				)
+			)
+		)
+	)
+	(symbol
 		(lib_id "power:+3V3")
 		(at 208.28 168.91 90)
@@
 					(unit 1)
 				)
-			)
-		)
-	)
-	(symbol
-		(lib_id "power:GND")
-		(at 231.14 134.62 0)
-		(unit 1)
-		(body_style 1)
-		(exclude_from_sim no)
-		(in_bom yes)
-		(on_board yes)
-		(in_pos_files yes)
-		(dnp no)
-		(fields_autoplaced yes)
-		(property "Reference" "#PWR061"
-			(at 231.14 140.97 0)
-			(hide yes)
-			(show_name no)
-			(do_not_autoplace no)
-			(effects
-				(font
-					(size 1.27 1.27)
-				)
-			)
-		)
-		(property "Value" "GND"
-			(at 231.14 138.7531 0)
-			(show_name no)
-			(do_not_autoplace no)
-			(effects
-				(font
-					(size 1.27 1.27)
-				)
-			)
-		)
-		(property "Footprint" ""
-			(at 231.14 134.62 0)
-			(hide yes)
-			(show_name no)
-			(do_not_autoplace no)
-			(effects
-				(font
-					(size 1.27 1.27)
-				)
-			)
-		)
-		(property "Datasheet" ""
-			(at 231.14 134.62 0)
-			(hide yes)
-			(show_name no)
-			(do_not_autoplace no)
-			(effects
-				(font
-					(size 1.27 1.27)
-				)
-			)
-		)
-		(property "Description" "Power symbol creates a global label with name \"GND\" , ground"
-			(at 231.14 134.62 0)
-			(hide yes)
-			(show_name no)
-			(do_not_autoplace no)
-			(effects
-				(font
-					(size 1.27 1.27)
-				)
-			)
-		)
-		(pin "1"
-		)
-		(instances
-			(project "battery-node"
-				(path "/0531bb65-44fe-462a-8fbf-92fb22c9abe0/a0e287d3-b915-410a-86a7-dfb59e4205a2"
-					(reference "#PWR061")
-					(unit 1)
-				)
