File: bms-logic/battery-node.kicad_pcb (KiCad board)
At the start: 4 copper layers, 44.2 x 66.4 mm, 219 parts, among them CN1 S12B-ZR-SM4A-TF, CN2 S4B-ZR-SM4A-TF_LF_SN, CN3 S4B-ZR-SM4A-TF_LF_SN, CN5 S4B-ZR-SM4A-TF_LF_SN, J3 Connector, USB-TYPE-C-16P, Q1 PBSS4350T,215, Q10 PBSS4350T,215, Q11 PBSS4350T,215, Q12 PBSS4350T,215, Q13 PBSS4350T,215, Q14 PBSS4350T,215, Q15 PBSS4350T,215, Q16 PBSS4350T,215, Q17 PBSS4350T,215, Q18 PBSS4350T,215, Q19 PBSS4350T,215, Q2 BSS123, Q3 DMZ6012E, Q4 DMZ6012E, Q5 PBSS4350T,215, Q6 PBSS4350T,215, Q7 PBSS4350T,215, Q8 PBSS4350T,215, Q9 PBSS4350T,215, U1 ESP32-H2-MINI-1-H2S, U10 ADUM3160, U11 LTV-217-B-G, U12 TCAN334D, U2 S8B-ZR-SM4A-TF_LF_SN, U4 BQ76972PFBR, U5 2SC2383_C41375137, U6 XC6206P332MR, U7 MP9485GN-Z, U8 MIE1W0505BGLVH-3R-Z, U9 ISO7041FDBQ

Commit message: cartesian
Parts:
- moved R15 56.7 mm to (75.9, 44.6), turned to -90 degrees
- moved D5 8.13 mm to (73.8, 45.6)
Routing:
- net /AFE/Cell16: track 56.0 -> 53.3 mm, vias 2 -> 3
Changed lines of the file:
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@@
 	(footprint "PCM_JLCPCB:R_0603"
 		(layer "F.Cu")
-		(at 131.445 56.388)
+		(at 75.946 44.577 -90)
 		(descr "Resistor SMD 0603 (1608 Metric), square (rectangular) end terminal, IPC_7351 nominal, (Body size source: IPC-SM-782 page 72, https://www.pcb-3d.com/wordpress/wp-content/uploads/ipc-sm-782a_amendment_1_and_2.pdf), generated with kicad-footprint-generator")
 		(tags "resistor")
 		(property "Reference" "R15"
-			(at 0 -1.3 0)
+			(at 0 -1.3 90)
 			(layer "F.SilkS")
 			(effects
@@
 		)
 		(property "Value" "15kΩ"
-			(at 0 1.43 0)
+			(at 0 1.43 90)
 			(layer "F.Fab")
 			(effects
@@
 		)
 		(property "Datasheet" "https://www.lcsc.com/datasheet/lcsc_datasheet_2206010130_UNI-ROYAL-Uniroyal-Elec-0603WAF1502T5E_C22809.pdf"
-			(at 0 0 0)
+			(at 0 0 270)
 			(unlocked yes)
 			(layer "F.Fab")
@@
 		)
 		(property "Description" "-55°C~+155°C 100mW 15kΩ 75V Thick Film Resistor ±1% ±100ppm/°C 0603 Chip Resistor - Surface Mount ROHS"
-			(at 0 0 0)
+			(at 0 0 270)
 			(unlocked yes)
 			(layer "F.Fab")
@@
 		)
 		(property "LCSC" "C22809"
-			(at 0 0 0)
+			(at 0 0 270)
 			(unlocked yes)
 			(layer "F.Fab")
@@
 		)
 		(property "Stock" "2155240"
-			(at 0 0 0)
+			(at 0 0 270)
 			(unlocked yes)
 			(layer "F.Fab")
@@
 		)
 		(property "Price" "0.005USD"
-			(at 0 0 0)
+			(at 0 0 270)
 			(unlocked yes)
 			(layer "F.Fab")
@@
 		)
 		(property "Process" "SMT"
-			(at 0 0 0)
+			(at 0 0 270)
 			(unlocked yes)
 			(layer "F.Fab")
@@
 		)
 		(property "Minimum Qty" "20"
-			(at 0 0 0)
+			(at 0 0 270)
 			(unlocked yes)
 			(layer "F.Fab")
@@
 		)
 		(property "Attrition Qty" "10"
-			(at 0 0 0)
+			(at 0 0 270)
 			(unlocked yes)
 			(layer "F.Fab")
@@
 		)
 		(property "Class" "Basic Component"
-			(at 0 0 0)
+			(at 0 0 270)
 			(unlocked yes)
 			(layer "F.Fab")
@@
 		)
 		(property "Category" "Resistors,Chip Resistor - Surface Mount"
-			(at 0 0 0)
+			(at 0 0 270)
 			(unlocked yes)
 			(layer "F.Fab")
@@
 		)
 		(property "Manufacturer" "UNI-ROYAL(Uniroyal Elec)"
-			(at 0 0 0)
+			(at 0 0 270)
 			(unlocked yes)
 			(layer "F.Fab")
@@
 		)
 		(property "Part" "0603WAF1502T5E"
-			(at 0 0 0)
+			(at 0 0 270)
 			(unlocked yes)
 			(layer "F.Fab")
@@
 		)
 		(property "Resistance" "15kΩ"
-			(at 0 0 0)
+			(at 0 0 270)
 			(unlocked yes)
 			(layer "F.Fab")
@@
 		)
 		(property "Power(Watts)" "100mW"
-			(at 0 0 0)
+			(at 0 0 270)
 			(unlocked yes)
 			(layer "F.Fab")
@@
 		)
 		(property "Type" "Thick Film Resistors"
-			(at 0 0 0)
+			(at 0 0 270)
 			(unlocked yes)
 			(layer "F.Fab")
@@
 		)
 		(property "Overload Voltage (Max)" "75V"
-			(at 0 0 0)
+			(at 0 0 270)
 			(unlocked yes)
 			(layer "F.Fab")
@@
 		)
 		(property "Operating Temperature Range" "-55°C~+155°C"
-			(at 0 0 0)
+			(at 0 0 270)
 			(unlocked yes)
 			(layer "F.Fab")
@@
 		)
 		(property "Tolerance" "±1%"
-			(at 0 0 0)
+			(at 0 0 270)
 			(unlocked yes)
 			(layer "F.Fab")
@@
 		)
 		(property "Temperature Coefficient" "±100ppm/°C"
-			(at 0 0 0)
+			(at 0 0 270)
 			(unlocked yes)
 			(layer "F.Fab")
@@
 		(duplicate_pad_numbers_are_jumpers no)
 		(fp_line
-			(start -1.3 -0.6)
-			(end 1.3 -0.6)
+			(start -1.3 0.6)
+			(end -1.3 -0.6)
 			(stroke
 				(width 0.05)
@@
 		)
 		(fp_line
-			(start -1.3 0.6)
-			(end -1.3 -0.6)
+			(start 1.3 0.6)
+			(end -1.3 0.6)
 			(stroke
 				(width 0.05)
@@
 		)
 		(fp_line
-			(start 1.3 -0.6)
-			(end 1.3 0.6)
+			(start -1.3 -0.6)
+			(end 1.3 -0.6)
 			(stroke
 				(width 0.05)
@@
 		)
 		(fp_line
-			(start 1.3 0.6)
-			(end -1.3 0.6)
+			(start 1.3 -0.6)
+			(end 1.3 0.6)
 			(stroke
 				(width 0.05)
@@
 		)
 		(fp_line
-			(start -0.8 -0.41)
-			(end 0.8 -0.41)
+			(start -0.8 0.41)
+			(end -0.8 -0.41)
 			(stroke
 				(width 0.1)
@@
 		)
 		(fp_line
-			(start -0.8 0.41)
-			(end -0.8 -0.41)
+			(start 0.8 0.41)
+			(end -0.8 0.41)
 			(stroke
 				(width 0.1)
@@
 		)
 		(fp_line
-			(start 0.8 -0.41)
-			(end 0.8 0.41)
+			(start -0.8 -0.41)
+			(end 0.8 -0.41)
 			(stroke
 				(width 0.1)
@@
 		)
 		(fp_line
-			(start 0.8 0.41)
-			(end -0.8 0.41)
+			(start 0.8 -0.41)
+			(end 0.8 0.41)
 			(stroke
 				(width 0.1)
@@
 		)
 		(fp_text user "${REFERENCE}"
-			(at 0 0 0)
+			(at 0 0 90)
 			(layer "F.Fab")
 			(effects
@@
 		)
 		(pad "1" smd roundrect
-			(at -0.82 0)
+			(at -0.82 0 270)
 			(size 0.8 0.95)
 			(layers "F.Cu" "F.Mask" "F.Paste")
@@
 		)
 		(pad "2" smd roundrect
-			(at 0.82 0)
+			(at 0.82 0 270)
 			(size 0.8 0.95)
 			(layers "F.Cu" "F.Mask" "F.Paste")
@@
 	(footprint "PCM_JLCPCB:D_SOD-123"
 		(layer "B.Cu")
-		(at 69.723 38.55598 90)
+		(at 73.787 45.593 90)
 		(descr "SOD-123")
 		(tags "SOD-123")
@@
 	)
 	(segment
+		(start 49.657 21.175624)
+		(end 49.657 22.86)
+		(width 0.508)
+		(layer "F.Cu")
+		(net "/AFE/Cell16")
+	)
+	(segment
 		(start 46.925 65.024)
 		(end 46.99 65.089)
@@
 	)
 	(segment
+		(start 50.8855 19.947124)
+		(end 49.657 21.175624)
+		(width 0.508)
+		(layer "F.Cu")
+		(net "/AFE/Cell16")
+	)
+	(segment
 		(start 51.68332 19.149304)
 		(end 50.8855 19.947124)
@@
 		(net "/AFE/Cell16")
 	)
+	(via
+		(at 49.657 22.86)
+		(size 0.6)
+		(drill 0.3)
+		(layers "F.Cu" "B.Cu")
+		(net "/AFE/Cell16")
+	)
 	(segment
 		(start 54.029 18.334)
@@
 	)
 	(segment
-		(start 52.451 19.370319)
-		(end 52.451 26.67)
-		(width 0.508)
-		(layer "In2.Cu")
-		(net "/AFE/Cell16")
-	)
-	(segment
-		(start 53.487319 18.334)
-		(end 52.451 19.370319)
+		(start 47.244 62.865)
+		(end 47.244 31.877)
 		(width 0.508)
 		(layer "In2.Cu")
@@
 	)
 	(segment
-		(start 52.451 26.67)
-		(end 47.244 31.877)
+		(start 45.085 65.024)
+		(end 47.244 62.865)
 		(width 0.508)
 		(layer "In2.Cu")
@@
 	)
 	(segment
-		(start 47.244 62.865)
-		(end 45.085 65.024)
+		(start 47.244 31.877)
+		(end 49.657 29.464)
 		(width 0.508)
 		(layer "In2.Cu")
@@
 	)
 	(segment
-		(start 47.244 31.877)
-		(end 47.244 62.865)
+		(start 49.657 29.464)
+		(end 49.657 22.86)
 		(width 0.508)
 		(layer "In2.Cu")

Commit message: kicad 10.0.1 before update to .2
Parts:
- removed D17: BZT52C75, PCM_JLCPCB:D_SOD-123
- C1, D3: moved to B.Cu
- D16: value BZT52C75 -> SMAJ60CA; footprint PCM_JLCPCB:D_SOD-123 -> Diode_SMD:D_SMA
- moved C1 70.1 mm to (58.8, 79.5)
- moved D2 49.0 mm to (61.2, 63.1)
- moved D3 45.3 mm to (60.7, 59.3), turned to 180 degrees
- moved R41 0.65 mm to (81.4, 70.2)
- moved R36 0.63 mm to (81.4, 64.3)
- moved C27 0.50 mm to (69.1, 59.4)
- moved R38 0.50 mm to (71.1, 59.4)
- moved C5 0.43 mm to (67.3, 31.1)
- moved C4 0.43 mm to (68.2, 33.9)
- moved C6 0.43 mm to (63.5, 34.4)
- moved D16 0.43 mm to (64.1, 39.8)
- moved R19 0.43 mm to (63.6, 32.4)
- moved U9 0.38 mm to (73.5, 66.2)
- moved C54 0.25 mm to (79.5, 62.1)
- moved R40 0.20 mm to (67.7, 71.3)
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Connections:
- CN1 pad MP: (no net) -> GND
- CN2 pad MP: (no net) -> GND
- CN3 pad MP: (no net) -> GND
- CN5 pad MP: (no net) -> GNDISO
- D16 pad 1: /AFE/AFE_BAT -> GND
- D16 pad 2: Net-(D16-Pad2) -> /AFE/AFE_BAT
- U2 pad MP: (no net) -> GND
Routing:
- net GNDISO: track 68.5 -> 25.2 mm, vias 15 -> 20
- net /AFE/Cell0: track 0.00 -> 10.4 mm, vias 0 -> 1
- net /AFE/VC6: track 15.5 -> 20.4 mm
- net /AFE/VC7: track 12.2 -> 17.2 mm
- net /AFE/VC8: track 8.27 -> 13.1 mm
- net /AFE/VC5: track 19.0 -> 23.4 mm
- net /AFE/VC0: track 40.8 -> 37.2 mm
- net /AFE/VC9: track 7.27 -> 10.4 mm
- net /AFE/VC16: track 33.0 -> 35.4 mm
- net /AFE/VC1: track 29.9 -> 32.4 mm
- net /AFE/VC11: track 14.3 -> 12.3 mm
- net /AFE/VC4: track 25.8 -> 27.7 mm
- net /AFE/VC10: track 10.7 -> 8.98 mm
- net GND: track 22.4 -> 23.7 mm, vias 24 -> 36
- net /AFE/VC12: track 17.8 -> 16.6 mm
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
Commit message: more layout, removed some unnecessary features
Parts:
- removed D11: BAT54C,215, PCM_JLCPCB:SOT-23-3_L2.9-W1.6-P1.90-LS2.8-BR
- removed D4: Red, PCM_JLCPCB:D_0603
- removed Q2: BSS123, PCM_JLCPCB:Q_SOT-23
- removed Q3, Q4: DMZ6012E, Package_TO_SOT_SMD:TSOT-23
- removed R15: 15kΩ, PCM_JLCPCB:R_0603
- removed R16: 100kΩ, PCM_JLCPCB:R_0402
- removed R17: 10kΩ, PCM_JLCPCB:R_0402
- removed R26, R27: 10kΩ, PCM_JLCPCB:R_0603
- removed TP18: IO8, TestPoint:TestPoint_Pad_D1.0mm
- added CN4: HX_JN1_27-2X10_TP_H4_9, JLCImport:HX_JN1_27-2X10_TP_H4_9, F.Cu at (80.3, 49.4)
- added CN6: HC-PBB08-2-20-F-H3.0-G1-R-P-04, easyeda2kicad:CONN-SMD_20P-P0.80_HC-PBB08-2-20-F-H4.0-G1-R-P-04, B.Cu at (79.0, 50.0)
- added D6: PMEG2010AEH_115, PCM_JLCPCB:D_SOD-123FL, B.Cu at (68.1, 51.0)
- added H1: MountingHole_Pad, MountingHole:MountingHole_2.2mm_M2_DIN965_Pad_TopBottom, F.Cu at (61.8, 20.2)
- added H2: MountingHole_Pad, MountingHole:MountingHole_2.2mm_M2_DIN965_Pad_TopBottom, F.Cu at (65.0, 58.9)
- added H3: MountingHole_Pad, MountingHole:MountingHole_2.2mm_M2_DIN965_Pad_TopBottom, F.Cu at (82.8, 72.6)
- added R90: 10kΩ, PCM_JLCPCB:R_0402, B.Cu at (65.5, 49.4)
- added TP24: IO8, TestPoint:TestPoint_Pad_D1.0mm, F.Cu at (19.6, 3.14)
- C13: moved to F.Cu
- C16, C8, D10, D12, D8, R20, R23, R24, R28, R29, R4: moved to B.Cu
- D7, D9: value BAT46W -> BAT41KFILM; footprint PCM_JLCPCB:D_SOD-123 -> PCM_JLCPCB:D_SOD-523; moved to B.Cu
- moved D12 56.6 mm to (61.2, 41.4), turned to 180 degrees
- moved C16 52.0 mm to (72.6, 38.5), turned to -45 degrees
- moved R4 51.8 mm to (72.8, 19.8)
- moved R28 49.7 mm to (68.6, 37.4), turned to 45 degrees
- moved C9 49.5 mm to (63.2, 56.4), turned to 45 degrees
- moved R29 49.4 mm to (69.6, 40.2), turned to 45 degrees
- moved C10 49.3 mm to (64.6, 55.0), turned to 45 degrees
- moved R20 47.6 mm to (64.8, 50.8), turned to -45 degrees
- moved R25 47.4 mm to (71.4, 39.4), turned to 180 degrees
- moved R22 46.6 mm to (70.4, 56.9), turned to 180 degrees
- moved C11 46.0 mm to (67.9, 57.4), turned to 90 degrees
- moved C12 45.9 mm to (68.9, 57.4), turned to 90 degrees
- moved C8 45.3 mm to (66.0, 52.7), turned to -45 degrees
- moved R21 45.2 mm to (70.4, 57.9), turned to 180 degrees
- moved U5 44.9 mm to (72.9, 35.9), turned to 90 degrees
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Connections:
- net /AFE/DCHG renamed /AFE/TEMP4
- net /AFE/DDSG renamed /AFE/TEMP3
- net Net-(U4-REG18) renamed /AFE/REG18
- net Net-(U4-SRN) renamed /AFE/SRN
- net Net-(U4-SRP) renamed /AFE/SRP
- C13 pad 1: Net-(D11-K) -> 5V0_SW
- C7 pad 1: /AFE/REG1_5V0 -> 3V3
- TP4 pad 1: Net-(U1-IO12) -> Net-(U1-IO0)
- TP7 pad 1: /CAN_SHUTDOWN -> Net-(U1-IO25/BOOT2)
- U1 pad 16: Net-(U1-IO12) -> /AFE/ALERT
- U1 pad 25: /CAN_SHUTDOWN -> Net-(U1-IO25/BOOT2)
- U1 pad 9: /AFE/ALERT -> Net-(U1-IO0)
- U4 pad 33: unconnected-(U4-RST_SHUT-Pad33) -> Net-(U4-RST_SHUT)
- U4 pad 35: /AFE/REG1_5V0 -> /AFE/REG1
- U6 pad 3: Net-(D11-K) -> 5V0_SW
- U9 pad 4: /CAN_SHUTDOWN -> unconnected-(U9-INB-Pad4)
Routing:
- net 5V0_SW: track 10.3 -> 61.1 mm, vias 6 -> 8
- net /CAN_RX: track 0.00 -> 44.8 mm, vias 0 -> 2
- net /CAN_TX: track 0.00 -> 43.9 mm, vias 0 -> 2
- net GND: track 23.7 -> 60.2 mm, vias 36 -> 67
- net /AFE/PACK: track 0.00 -> 36.2 mm, vias 0 -> 3
- net /USB_D-: track 2.99 -> 38.6 mm, vias 0 -> 1
- net /USB_D+: track 3.16 -> 38.6 mm, vias 0 -> 1
- net /AFE/LD: track 0.00 -> 34.6 mm, vias 0 -> 5
- net /AFE/CURRENT_SENSE_N: track 0.00 -> 22.4 mm, vias 0 -> 3
- net /AFE/PDSG_GATE_CTRL: track 0.00 -> 20.7 mm, vias 0 -> 2
- net /EN_ISO_PWR: track 4.14 -> 23.8 mm
- net /AFE/CURRENT_SENSE_P: track 0.00 -> 18.3 mm, vias 0 -> 3
- net /AFE/FUSE: track 0.00 -> 16.9 mm, vias 0 -> 2
- net 3V3: track 3.37 -> 18.4 mm, vias 3 -> 13
- net /AFE/REGIN: track 0.00 -> 13.8 mm
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- added copper zone on B.Cu, net /AFE/AFE_BAT
- added copper zone on B.Cu, net Net-(D12-Pad1)
Other:
- board size 44.2 x 66.4 mm -> 44.2 x 66.5 mm
