File: bms-logic/battery-node.kicad_pcb (KiCad board)
At the start: 4 copper layers, 44.2 x 66.5 mm, 215 parts, among them CN1 S12B-ZR-SM4A-TF, CN2 S4B-ZR-SM4A-TF_LF_SN, CN3 S4B-ZR-SM4A-TF_LF_SN, CN4 HX_JN1_27-2X10_TP_H4_9, CN5 S4B-ZR-SM4A-TF_LF_SN, CN6 HC-PBB08-2-20-F-H3.0-G1-R-P-04, J3 Connector, USB-TYPE-C-16P, Q1 PBSS4350T,215, Q10 PBSS4350T,215, Q11 PBSS4350T,215, Q12 PBSS4350T,215, Q13 PBSS4350T,215, Q14 PBSS4350T,215, Q15 PBSS4350T,215, Q16 PBSS4350T,215, Q17 PBSS4350T,215, Q18 PBSS4350T,215, Q19 PBSS4350T,215, Q5 PBSS4350T,215, Q6 PBSS4350T,215, Q7 PBSS4350T,215, Q8 PBSS4350T,215, Q9 PBSS4350T,215, U1 ESP32-H2-MINI-1-H2S, U10 ADUM3160, U11 LTV-217-B-G, U12 TCAN334D, U2 S8B-ZR-SM4A-TF_LF_SN, U4 BQ76972PFBR, U5 2SC2383_C41375137, U6 XC6206P332MR, U7 MP9485GN-Z, U8 MIE1W0505BGLVH-3R-Z, U9 ISO7041FDBQ

Commit message: done with layout, need to address some DRC
Parts:
- removed TP6: IO25, TestPoint:TestPoint_Pad_D1.0mm
- added C52: 470pF, PCM_JLCPCB:C_0402, B.Cu at (70.1, 53.2)
- added C53: 470pF, PCM_JLCPCB:C_0402, B.Cu at (69.4, 53.9)
- C50, C51, C56, C57, C7, R1, R2, TP1, TP12, TP13, TP14, TP16, TP17, TP19, TP2, TP23, TP3, TP4, TP5, TP7: moved to B.Cu
- LED1: value MHT136UBCT -> ~
- moved TP11 81.3 mm to (76.3, 57.7)
- moved TP17 81.1 mm to (76.7, 33.3)
- moved TP19 77.6 mm to (76.5, 28.4)
- moved TP16 75.0 mm to (71.7, 26.1)
- moved TP1 71.9 mm to (75.4, 20.1)
- moved TP24 71.7 mm to (71.6, 52.6)
- moved TP3 70.6 mm to (74.8, 23.4)
- moved TP5 69.6 mm to (74.6, 27.5)
- moved TP12 67.4 mm to (59.2, 23.9)
- moved TP2 65.1 mm to (68.7, 21.9)
- moved TP8 64.0 mm to (69.6, 32.3)
- moved TP7 63.4 mm to (69.1, 29.0)
- moved TP4 63.2 mm to (68.0, 23.8)
- moved TP9 60.8 mm to (67.6, 32.3)
- moved R3 57.3 mm to (66.1, 22.0), turned to -90 degrees
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- renumbered U2 to CN2, CN2 to CN4, CN4 to CN5, CN5 to CN7, J3 to CN8
Connections:
- net /AFE/CHG_GATE_CTRL renamed /AFE/CHG_GATE_CONTROL
- C7 pad 1: 3V3 -> /AFE/REG1
- CN5 pad 1: /AFE/DSG_GATE_CONTROL -> /AFE/CHARGE_PUMP
- CN5 pad 10: /AFE/TEMP_DSG -> /AFE/TEMP_DSG_FETS
- CN5 pad 5: /AFE/CHARGE_PUMP -> /AFE/DSG_GATE_CONTROL
- CN5 pad 6: /AFE/FUSE -> unconnected-(CN5-Pad6)
- CN5 pad 8: /AFE/TEMP_CHG -> /AFE/TEMP_CHG_FETS
- CN6 pad 12: /AFE/TEMP_DSG -> /AFE/TEMP_DSG_FETS
- CN6 pad 14: /AFE/TEMP_CHG -> /AFE/TEMP_CHG_FETS
- CN6 pad 15: /AFE/CHARGE_PUMP -> /AFE/DSG_GATE_CONTROL
- CN6 pad 16: /AFE/FUSE -> unconnected-(CN6-Pad16)
- CN6 pad 19: /AFE/DSG_GATE_CONTROL -> /AFE/CHARGE_PUMP
- TP4 pad 1: Net-(U1-IO0) -> Net-(U1-IO5/ADC/MTDI)
- TP9 pad 1: /CAN_SLEEP -> Net-(U1-IO8/BOOT0)
- U1 pad 10: /AFE/nWAKE -> /HEARTBEAT_LED
- U1 pad 16: /AFE/ALERT -> /CAN_TX
- U1 pad 19: /HEARTBEAT_LED -> Net-(U1-IO5/ADC/MTDI)
- U1 pad 21: /CAN_TX -> /AFE/ALERT
- U1 pad 22: /CAN_SLEEP -> Net-(U1-IO8/BOOT0)
- U1 pad 30: Net-(U1-IO23/RXD0) -> /CAN_SLEEP
- U1 pad 9: Net-(U1-IO0) -> /AFE/nWAKE
- U4 pad 21: /AFE/TEMP1 -> /AFE/TEMP_CELLS_4
- U4 pad 23: /AFE/TEMP2 -> /AFE/TEMP_CELLS_3
- U4 pad 31: /AFE/TEMP4 -> /AFE/TEMP_CELLS_1
- U4 pad 32: /AFE/TEMP3 -> /AFE/TEMP_CELLS_2
Routing:
- net /AFE/SDA: track 0.00 -> 61.0 mm, vias 0 -> 2
- net /USB_nINT: track 3.24 -> 60.9 mm, vias 1 -> 4
- net /AFE/TEMP_CELLS_2: track 0.00 -> 55.3 mm, vias 0 -> 3
- net /AFE/TEMP_CELLS_1: track 0.00 -> 51.8 mm, vias 0 -> 3
- net /AFE/ALERT: track 0.00 -> 49.2 mm, vias 0 -> 2
- net /AFE/SDL: track 0.00 -> 49.2 mm, vias 0 -> 2
- net /EN_ISO_PWR: track 23.8 -> 72.3 mm, vias 0 -> 3
- net /AFE/nWAKE: track 2.40 -> 50.5 mm, vias 1 -> 3
- net /AFE/TEMP_CELLS_4: track 0.00 -> 39.2 mm, vias 0 -> 2
- net /CAN_SLEEP: track 0.00 -> 39.0 mm, vias 0 -> 2
- net /AFE/TEMP_CELLS_3: track 0.00 -> 37.7 mm, vias 0 -> 2
- net /AFE/CHG_GATE_CONTROL: track 6.60 -> 27.0 mm, vias 2 -> 3
- net /AFE/CHARGE_PUMP: track 9.63 -> 29.8 mm, vias 2 -> 3
- net GND: track 60.2 -> 80.1 mm, vias 67 -> 76
- net /AFE/DSG_GATE_CONTROL: track 6.86 -> 25.0 mm, vias 2 -> 3
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- added copper zone on B.Cu, net Net-(U5-C)
- added copper zone on F.Cu, net Net-(U5-C)
Other:
- outline, holes or cut-outs redrawn
- board text added: "+"
- board text added: "-"
- board text added: "0"
- board text added: "1"
- board text added: "10"
- board text added: "11"
- board text added: "12"
- board text added: "13"
- board text added: "14"
- board text added: "15"
- board text added: "16"
- board text added: "2"
- board text added: "3"
- board text added: "4"
- board text added: "5"
- board text added: "51026"
- board text added: "6"
- board text added: "7"
- board text added: "8"
- board text added: "9"
- board text added: "CDT"
- board text added: "HVBMS Rev-A"
- board text added: "T1"
- board text added: "T2"
- board text added: "T3"
- board text added: "T4"
