File: bms-logic/battery-node.kicad_sch (KiCad schematic)
At the start: 25 parts, among them J1 TC2050, U1 ESP32-H2-MINI-1-H2S

Commit message: started afe layout
Parts:
- J1, R10, R5, R6, R7, R8, R9: now fitted
- JP1: now fitted; now left out of the parts list
Connections:
- net +3V3: no longer R1.2, R2.2, R4.2, TP10.1, U1.3 (3V3)
- new net 3V3: R1.2, R2.2, R4.2, TP10.1, U1.3 (3V3)
Changed lines of the file:
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@@
 		)
 	)
+	(rule_area
+		(exclude_from_sim no)
+		(in_bom no)
+		(on_board no)
+		(dnp yes)
+		(polyline
+			(pts
+				(xy 295.91 198.12) (xy 295.91 262.89) (xy 172.72 262.89) (xy 172.72 198.12)
+			)
+			(stroke
+				(width 0)
+				(type dash)
+			)
+			(fill
+				(type color)
+				(color 0 0 0 0.1490196078)
+			)
+		)
+	)
 	(symbol
 		(lib_id "Connector:TestPoint")
@@
 			)
 		)
-		(property "Value" "+3V3"
-			(at 127 171.7731 0)
+		(property "Value" "3V3"
+			(at 125.603 168.91 0)
 			(show_name no)
 			(do_not_autoplace no)
@@
 					(size 1.27 1.27)
 				)
+				(justify right)
 			)
 		)
@@
 		(exclude_from_sim no)
 		(in_bom yes)
-		(on_board no)
+		(on_board yes)
 		(in_pos_files yes)
-		(dnp yes)
+		(dnp no)
 		(fields_autoplaced yes)
 		(property "Reference" "R7"
@@
 		(body_style 1)
 		(exclude_from_sim no)
-		(in_bom yes)
-		(on_board no)
+		(in_bom no)
+		(on_board yes)
 		(in_pos_files yes)
-		(dnp yes)
+		(dnp no)
 		(fields_autoplaced yes)
 		(property "Reference" "JP1"
@@
 			)
 		)
-		(property "Value" "+3V3"
-			(at 241.3 147.955 90)
+		(property "Value" "3V3"
+			(at 239.903 146.05 0)
 			(show_name no)
 			(do_not_autoplace no)
@@
 					(size 1.27 1.27)
 				)
-				(justify left)
+				(justify right)
 			)
 		)
@@
 		(exclude_from_sim no)
 		(in_bom no)
-		(on_board no)
+		(on_board yes)
 		(in_pos_files yes)
-		(dnp yes)
+		(dnp no)
 		(fields_autoplaced yes)
 		(property "Reference" "J1"
@@
 		(exclude_from_sim no)
 		(in_bom yes)
-		(on_board no)
+		(on_board yes)
 		(in_pos_files yes)
-		(dnp yes)
+		(dnp no)
 		(fields_autoplaced yes)
 		(property "Reference" "R5"
@@
 		(exclude_from_sim no)
 		(in_bom yes)
-		(on_board no)
+		(on_board yes)
 		(in_pos_files yes)
-		(dnp yes)
+		(dnp no)
 		(fields_autoplaced yes)
 		(property "Reference" "R9"
@@
 			)
 		)
-		(property "Value" "+3V3"
-			(at 203.2 87.3069 0)
+		(property "Value" "3V3"
+			(at 204.597 90.17 0)
 			(show_name no)
 			(do_not_autoplace no)
@@
 					(size 1.27 1.27)
 				)
+				(justify left)
 			)
 		)
@@
 		(exclude_from_sim no)
 		(in_bom yes)
-		(on_board no)
+		(on_board yes)
 		(in_pos_files yes)
-		(dnp yes)
+		(dnp no)
 		(fields_autoplaced yes)
 		(property "Reference" "R10"
@@
 		(exclude_from_sim no)
 		(in_bom yes)
-		(on_board no)
+		(on_board yes)
 		(in_pos_files yes)
-		(dnp yes)
+		(dnp no)
 		(fields_autoplaced yes)
 		(property "Reference" "R6"
@@
 		(exclude_from_sim no)
 		(in_bom yes)
-		(on_board no)
+		(on_board yes)
 		(in_pos_files yes)
-		(dnp yes)
+		(dnp no)
 		(fields_autoplaced yes)
 		(property "Reference" "R8"

Commit message: power supply layout
Parts:
- added JP5: SolderJumper_2_Open, Jumper:SolderJumper-2_P1.3mm_Open_RoundedPad1.0x1.5mm, symbol Jumper:SolderJumper_2_Open
- added R33: 100kΩ, PCM_JLCPCB:R_0402, symbol PCM_JLCPCB-Resistors:0402,100kΩ
- added TP23: IO25, TestPoint:TestPoint_Pad_D1.0mm, symbol Connector:TestPoint
Connections:
- net 3V3: now also JP5.2 (B)
- net GND: now also R33.2
- net at U1.24 (IO22): now also TP23.1
- net ISOLATED_COMMS/CAN_SHUTDOWN renamed CAN_SHUTDOWN
- net ISOLATED_COMMS/CAN_SLEEP renamed CAN_SLEEP
- net ISOLATED_COMMS/EN_ISO_PWR renamed EN_ISO_PWR
- net EN_ISO_PWR: now also JP5.1 (A), R33.1
- net ISOLATED_COMMS/USB_D+ renamed USB_D+
- net ISOLATED_COMMS/USB_D- renamed USB_D-
- net ISOLATED_COMMS/USB_nINT renamed USB_nINT
Other:
- note added: "Jump to force enable (first time flashing)"
- note added: "On: HIGH Off: LOW"

Commit message: diagonal
Parts:
- added H1, H2: MountingHole_Pad, symbol Mechanical:MountingHole_Pad
Connections:
- no-connect marks 2 -> 4
Changed lines of the file:
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@@
 	)
 	(no_connect
+		(at 251.46 64.77)
+	)
+	(no_connect
 		(at 200.66 97.79)
 	)
@@
 		(at 240.03 237.49)
 	)
+	(no_connect
+		(at 251.46 69.85)
+	)
 	(wire
 		(pts
@@
 	)
 	(symbol
+		(lib_id "Mechanical:MountingHole_Pad")
+		(at 248.92 69.85 90)
+		(unit 1)
+		(body_style 1)
+		(exclude_from_sim no)
+		(in_bom no)
+		(on_board yes)
+		(in_pos_files yes)
+		(dnp no)
+		(property "Reference" "H1"
+			(at 235.204 68.1877 90)
+			(show_name no)
+			(do_not_autoplace no)
+			(effects
+				(font
+					(size 1.27 1.27)
+				)
+			)
+		)
+		(property "Value" "MountingHole_Pad"
+			(at 235.204 70.612 90)
+			(show_name no)
+			(do_not_autoplace no)
+			(effects
+				(font
+					(size 1.27 1.27)
+				)
+			)
+		)
+		(property "Footprint" ""
+			(at 248.92 69.85 0)
+			(hide yes)
+			(show_name no)
+			(do_not_autoplace no)
+			(effects
+				(font
+					(size 1.27 1.27)
+				)
+			)
+		)
+		(property "Datasheet" ""
+			(at 248.92 69.85 0)
+			(hide yes)
+			(show_name no)
+			(do_not_autoplace no)
+			(effects
+				(font
+					(size 1.27 1.27)
+				)
+			)
+		)
+		(property "Description" "Mounting Hole with connection"
+			(at 248.92 69.85 0)
+			(hide yes)
+			(show_name no)
+			(do_not_autoplace no)
+			(effects
+				(font
+					(size 1.27 1.27)
+				)
+			)
+		)
+		(pin "1"
+		)
+		(instances
+			(project "battery-node"
+				(path "/0531bb65-44fe-462a-8fbf-92fb22c9abe0"
+					(reference "H1")
+					(unit 1)
+				)
+			)
+		)
+	)
+	(symbol
 		(lib_id "PCM_JLCPCB-Resistors:0402,33Ω")
 		(at 256.54 219.71 270)
@@
 					(unit 1)
 				)
+			)
+		)
+	)
+	(symbol
+		(lib_id "Mechanical:MountingHole_Pad")
+		(at 248.92 64.77 90)
+		(unit 1)
+		(body_style 1)
+		(exclude_from_sim no)
+		(in_bom no)
+		(on_board yes)
+		(in_pos_files yes)
+		(dnp no)
+		(property "Reference" "H2"
+			(at 236.22 62.3457 90)
+			(show_name no)
+			(do_not_autoplace no)
+			(effects
+				(font
+					(size 1.27 1.27)
+				)
+			)
+		)
+		(property "Value" "MountingHole_Pad"
+			(at 236.22 64.77 90)
+			(show_name no)
+			(do_not_autoplace no)
+			(effects
+				(font
+					(size 1.27 1.27)
+				)
+			)
+		)
+		(property "Footprint" ""
+			(at 248.92 64.77 0)
+			(hide yes)
+			(show_name no)
+			(do_not_autoplace no)
+			(effects
+				(font
+					(size 1.27 1.27)
+				)
+			)
+		)
+		(property "Datasheet" ""
+			(at 248.92 64.77 0)
+			(hide yes)
+			(show_name no)
+			(do_not_autoplace no)
+			(effects
+				(font
+					(size 1.27 1.27)
+				)
+			)
+		)
+		(property "Description" "Mounting Hole with connection"
+			(at 248.92 64.77 0)
+			(hide yes)
+			(show_name no)
+			(do_not_autoplace no)
+			(effects
+				(font
+					(size 1.27 1.27)
+				)
+			)
+		)
+		(pin "1"
+		)
+		(instances
+			(project "battery-node"
+				(path "/0531bb65-44fe-462a-8fbf-92fb22c9abe0"
+					(reference "H2")
+					(unit 1)
+				)

Commit message: kicad 10.0.1 before update to .2
Other:
- note added: "Add interface for display"
Changed lines of the file:
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@@
+		)
+	)
+	(text "Add interface for display"
+		(exclude_from_sim no)
+		(at 183.134 82.296 0)
+		(effects
+			(font
+				(size 1.27 1.27)
+			)
 		)
 	)

Commit message: more layout, removed some unnecessary features
Parts:
- added H3: MountingHole_Pad, MountingHole:MountingHole_2.2mm_M2_DIN965_Pad_TopBottom, symbol Mechanical:MountingHole_Pad
- H1, H2: footprint (none) -> MountingHole:MountingHole_2.2mm_M2_DIN965_Pad_TopBottom
Connections:
- net AFE/ALERT: now also U1.16 (IO12); no longer U1.9 (IO0)
- net at TP4.1: now also U1.9 (IO0); no longer U1.16 (IO12)
- net CAN_SHUTDOWN: no longer names the net of TP7.1, U1.25 (IO25/BOOT2)
- no-connect marks 4 -> 5
Other:
- sheet ISOLATED_COMMS ports: added none; removed CAN_SHUTDOWN
- note added: "Deep sleep wakeup pins: IO 8-14"
- note added: "No decoupling cap needed; implemented on ESP32 subcircuit"

Commit message: done with layout, need to address some DRC
Parts:
- removed TP6: IO25, TestPoint:TestPoint_Pad_D1.0mm, symbol Connector:TestPoint
Connections:
- net AFE/ALERT: now also U1.21 (IO11); no longer U1.16 (IO12)
- net AFE/nWAKE: now also U1.9 (IO0); no longer U1.10 (IO1/ADC)
- net CAN_SLEEP: now also U1.30 (IO23/RXD0); no longer TP9.1, U1.22 (IO8/BOOT0)
- net CAN_TX: now also U1.16 (IO12); no longer U1.21 (IO11)
- net HEARTBEAT_LED: now also U1.10 (IO1/ADC); no longer U1.19 (IO5/ADC/MTDI)
- net at TP4.1: now also U1.19 (IO5/ADC/MTDI); no longer U1.9 (IO0)
- new net: TP9.1, U1.22 (IO8/BOOT0)
