File: bms-logic/thermistor.kicad_sch (KiCad schematic)
At the start: 2 parts, among them CN1 A2001WR-S-2P

Commit message: started afe layout
Parts:
- renumbered C6 to C50
Changed lines of the file:
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@@
 		(dnp no)
 		(fields_autoplaced yes)
-		(property "Reference" "#PWR078"
+		(property "Reference" "#PWR074"
 			(at 111.76 106.68 0)
 			(hide yes)
@@
 			(project "battery-node"
 				(path "/0531bb65-44fe-462a-8fbf-92fb22c9abe0/2e6fa66d-cf61-4130-94fd-f989bd2a39c4/14facb8c-7913-48f0-8c95-94965f8c72e2"
-					(reference "#PWR085")
+					(reference "#PWR082")
 					(unit 1)
 				)
 				(path "/0531bb65-44fe-462a-8fbf-92fb22c9abe0/2e6fa66d-cf61-4130-94fd-f989bd2a39c4/524a3c24-e1d4-440c-a5de-5fa78cca8f92"
-					(reference "#PWR081")
+					(reference "#PWR078")
 					(unit 1)
 				)
 				(path "/0531bb65-44fe-462a-8fbf-92fb22c9abe0/2e6fa66d-cf61-4130-94fd-f989bd2a39c4/5ed4f55b-1488-4427-9d20-f9a6669b64e7"
-					(reference "#PWR078")
+					(reference "#PWR074")
 					(unit 1)
 				)
 				(path "/0531bb65-44fe-462a-8fbf-92fb22c9abe0/2e6fa66d-cf61-4130-94fd-f989bd2a39c4/a9e3e829-22d3-464f-b954-379e2fb6907f"
-					(reference "#PWR089")
+					(reference "#PWR086")
 					(unit 1)
 				)
@@
 		(dnp no)
 		(fields_autoplaced yes)
-		(property "Reference" "#PWR079"
+		(property "Reference" "#PWR073"
 			(at 111.76 76.2 0)
 			(hide yes)
@@
 			(project "battery-node"
 				(path "/0531bb65-44fe-462a-8fbf-92fb22c9abe0/2e6fa66d-cf61-4130-94fd-f989bd2a39c4/14facb8c-7913-48f0-8c95-94965f8c72e2"
-					(reference "#PWR084")
+					(reference "#PWR081")
 					(unit 1)
 				)
 				(path "/0531bb65-44fe-462a-8fbf-92fb22c9abe0/2e6fa66d-cf61-4130-94fd-f989bd2a39c4/524a3c24-e1d4-440c-a5de-5fa78cca8f92"
-					(reference "#PWR080")
+					(reference "#PWR077")
 					(unit 1)
 				)
 				(path "/0531bb65-44fe-462a-8fbf-92fb22c9abe0/2e6fa66d-cf61-4130-94fd-f989bd2a39c4/5ed4f55b-1488-4427-9d20-f9a6669b64e7"
-					(reference "#PWR079")
+					(reference "#PWR073")
 					(unit 1)
 				)
 				(path "/0531bb65-44fe-462a-8fbf-92fb22c9abe0/2e6fa66d-cf61-4130-94fd-f989bd2a39c4/a9e3e829-22d3-464f-b954-379e2fb6907f"
-					(reference "#PWR088")
+					(reference "#PWR085")
 					(unit 1)
 				)
@@
 		(dnp no)
 		(fields_autoplaced yes)
-		(property "Reference" "#PWR077"
+		(property "Reference" "#PWR075"
 			(at 123.19 104.14 0)
 			(hide yes)
@@
 			(project "battery-node"
 				(path "/0531bb65-44fe-462a-8fbf-92fb22c9abe0/2e6fa66d-cf61-4130-94fd-f989bd2a39c4/14facb8c-7913-48f0-8c95-94965f8c72e2"
-					(reference "#PWR086")
+					(reference "#PWR083")
 					(unit 1)
 				)
 				(path "/0531bb65-44fe-462a-8fbf-92fb22c9abe0/2e6fa66d-cf61-4130-94fd-f989bd2a39c4/524a3c24-e1d4-440c-a5de-5fa78cca8f92"
-					(reference "#PWR082")
+					(reference "#PWR079")
 					(unit 1)
 				)
 				(path "/0531bb65-44fe-462a-8fbf-92fb22c9abe0/2e6fa66d-cf61-4130-94fd-f989bd2a39c4/5ed4f55b-1488-4427-9d20-f9a6669b64e7"
-					(reference "#PWR077")
+					(reference "#PWR075")
 					(unit 1)
 				)
 				(path "/0531bb65-44fe-462a-8fbf-92fb22c9abe0/2e6fa66d-cf61-4130-94fd-f989bd2a39c4/a9e3e829-22d3-464f-b954-379e2fb6907f"
-					(reference "#PWR090")
+					(reference "#PWR087")
 					(unit 1)
 				)
@@
 		(dnp no)
 		(fields_autoplaced yes)
-		(property "Reference" "#PWR017"
+		(property "Reference" "#PWR076"
 			(at 135.89 104.14 0)
 			(hide yes)
@@
 			(project "battery-node"
 				(path "/0531bb65-44fe-462a-8fbf-92fb22c9abe0/2e6fa66d-cf61-4130-94fd-f989bd2a39c4/14facb8c-7913-48f0-8c95-94965f8c72e2"
-					(reference "#PWR087")
+					(reference "#PWR084")
 					(unit 1)
 				)
 				(path "/0531bb65-44fe-462a-8fbf-92fb22c9abe0/2e6fa66d-cf61-4130-94fd-f989bd2a39c4/524a3c24-e1d4-440c-a5de-5fa78cca8f92"
-					(reference "#PWR083")
+					(reference "#PWR080")
 					(unit 1)
 				)
 				(path "/0531bb65-44fe-462a-8fbf-92fb22c9abe0/2e6fa66d-cf61-4130-94fd-f989bd2a39c4/5ed4f55b-1488-4427-9d20-f9a6669b64e7"
-					(reference "#PWR017")
+					(reference "#PWR076")
 					(unit 1)
 				)
 				(path "/0531bb65-44fe-462a-8fbf-92fb22c9abe0/2e6fa66d-cf61-4130-94fd-f989bd2a39c4/a9e3e829-22d3-464f-b954-379e2fb6907f"
-					(reference "#PWR091")
+					(reference "#PWR088")
 					(unit 1)
 				)
@@
 		(in_pos_files yes)
 		(dnp no)
-		(property "Reference" "C6"
+		(property "Reference" "C50"
 			(at 137.16 92.71 90)
 			(show_name no)
@@
 			(project "battery-node"
 				(path "/0531bb65-44fe-462a-8fbf-92fb22c9abe0/2e6fa66d-cf61-4130-94fd-f989bd2a39c4/14facb8c-7913-48f0-8c95-94965f8c72e2"
-					(reference "C55")
+					(reference "C52")
 					(unit 1)
 				)
 				(path "/0531bb65-44fe-462a-8fbf-92fb22c9abe0/2e6fa66d-cf61-4130-94fd-f989bd2a39c4/524a3c24-e1d4-440c-a5de-5fa78cca8f92"
-					(reference "C54")
+					(reference "C51")
 					(unit 1)
 				)
 				(path "/0531bb65-44fe-462a-8fbf-92fb22c9abe0/2e6fa66d-cf61-4130-94fd-f989bd2a39c4/5ed4f55b-1488-4427-9d20-f9a6669b64e7"
-					(reference "C6")
+					(reference "C50")
 					(unit 1)
 				)
 				(path "/0531bb65-44fe-462a-8fbf-92fb22c9abe0/2e6fa66d-cf61-4130-94fd-f989bd2a39c4/a9e3e829-22d3-464f-b954-379e2fb6907f"
-					(reference "C56")
-					(unit 1)
-				)
+					(reference "C53")
+					(unit 1)
+				)

Commit message: isolated comms
Parts:
- removed CN1: A2001WR-S-2P, JLCImport:A2001WR-S-2P, symbol JLCImport:A2001WR-S-2P
- added P1: SM02B-NSHSS-TB_LF_SN, JLCImport:SM02B-NSHSS-TB_LF_SN, symbol JLCImport:SM02B-NSHSS-TB_LF_SN
Connections:
- net GND: now also P1.1, P1.3, P1.4
- net THERMISTOR_CHANNEL: now also P1.2
Other:
- note added: "use smaller connector"
Changed lines of the file:
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@@
 	(generator_version "10.0")
 	(paper "A4")
+	(text "use smaller connector"
+		(exclude_from_sim no)
+		(at 129.032 105.156 0)
+		(effects
+			(font
+				(size 1.27 1.27)
+			)
+		)
+	)
 	(junction
 		(at 135.89 90.17)
@@
 	(symbol
 		(lib_id "power:GND")
-		(at 111.76 100.33 0)
+		(at 111.76 97.79 0)
 		(unit 1)
 		(body_style 1)
@@
 		(fields_autoplaced yes)
 		(property "Reference" "#PWR074"
-			(at 111.76 106.68 0)
+			(at 111.76 104.14 0)
 			(hide yes)
 			(show_name no)
@@
 		)
 		(property "Value" "GND"
-			(at 111.76 104.4631 0)
+			(at 111.76 101.9231 0)
 			(show_name no)
 			(do_not_autoplace no)
@@
 		)
 		(property "Footprint" ""
-			(at 111.76 100.33 0)
+			(at 111.76 97.79 0)
 			(hide yes)
 			(show_name no)
@@
 		)
 		(property "Datasheet" ""
-			(at 111.76 100.33 0)
+			(at 111.76 97.79 0)
 			(hide yes)
 			(show_name no)
@@
 		)
 		(property "Description" "Power symbol creates a global label with name \"GND\" , ground"
-			(at 111.76 100.33 0)
+			(at 111.76 97.79 0)
 			(hide yes)
 			(show_name no)
@@
 	(symbol
 		(lib_id "power:GND")
-		(at 111.76 82.55 180)
+		(at 111.76 85.09 180)
 		(unit 1)
 		(body_style 1)
@@
 		(fields_autoplaced yes)
 		(property "Reference" "#PWR073"
-			(at 111.76 76.2 0)
+			(at 111.76 78.74 0)
 			(hide yes)
 			(show_name no)
@@
 		)
 		(property "Value" "GND"
-			(at 111.76 78.4169 0)
+			(at 111.76 80.9569 0)
 			(show_name no)
 			(do_not_autoplace no)
@@
 		)
 		(property "Footprint" ""
-			(at 111.76 82.55 0)
+			(at 111.76 85.09 0)
 			(hide yes)
 			(show_name no)
@@
 		)
 		(property "Datasheet" ""
-			(at 111.76 82.55 0)
+			(at 111.76 85.09 0)
 			(hide yes)
 			(show_name no)
@@
 		)
 		(property "Description" "Power symbol creates a global label with name \"GND\" , ground"
-			(at 111.76 82.55 0)
+			(at 111.76 85.09 0)
 			(hide yes)
 			(show_name no)
@@
 	)
 	(symbol
-		(lib_id "JLCImport:A2001WR-S-2P")
-		(at 115.57 91.44 180)
-		(unit 1)
-		(body_style 1)
-		(exclude_from_sim no)
-		(in_bom yes)
-		(on_board yes)
-		(in_pos_files yes)
-		(dnp no)
-		(fields_autoplaced yes)
-		(property "Reference" "CN1"
-			(at 108.458 90.2278 0)
-			(show_name no)
-			(do_not_autoplace no)
-			(effects
-				(font
-					(size 1.27 1.27)
-				)
-				(justify left)
-			)
-		)
-		(property "Value" "A2001WR-S-2P"
-			(at 108.458 92.6521 0)
-			(show_name no)
-			(do_not_autoplace no)
-			(effects
-				(font
-					(size 1.27 1.27)
-				)
-				(justify left)
-			)
-		)
-		(property "Footprint" "JLCImport:A2001WR-S-2P"
-			(at 115.57 91.44 0)
-			(hide yes)
-			(show_name no)
-			(do_not_autoplace no)
-			(effects
-				(font
-					(size 1.27 1.27)
-				)
-			)
-		)
-		(property "Datasheet" "https://www.lcsc.com/datasheet/lcsc_datasheet_2304140030_CJT-Changjiang-Connectors-A2001WR-S-2P_C225233.pdf"
-			(at 115.57 91.44 0)
-			(hide yes)
-			(show_name no)
-			(do_not_autoplace no)
-			(effects
-				(font
-					(size 1.27 1.27)
-				)
-			)
-		)
-		(property "Description" "-40℃~+105℃ 1 100V 1x2P 2 2A 2P 2mm LCP PH Phosphor Bronze Surface Mount, Right Angle Tin UL94V-0 SMD,P=2mm,卧贴 Wire To Board Connector ROHS"
-			(at 115.57 91.44 0)
-			(hide yes)
-			(show_name no)
-			(do_not_autoplace no)
-			(effects
-				(font
-					(size 1.27 1.27)
-				)
-			)
-		)
-		(property "LCSC" "C225233"
-			(at 115.57 91.44 0)
-			(hide yes)
-			(show_name no)
-			(do_not_autoplace no)
-			(effects
-				(font
-					(size 1.27 1.27)
-				)
-			)
-		)
-		(property "Manufacturer" "CJT(Changjiang Connectors)"
-			(at 115.57 91.44 0)
-			(hide yes)
-			(show_name no)
-			(do_not_autoplace no)
-			(effects
-				(font
-					(size 1.27 1.27)
-				)
-			)
-		)
-		(property "Manufacturer Part" "A2001WR-S-2P"
-			(at 115.57 91.44 0)
-			(hide yes)
-			(show_name no)
-			(do_not_autoplace no)
-			(effects
-				(font
-					(size 1.27 1.27)
-				)
-			)
-		)
-		(pin "1"
-		)
-		(pin "2"
-		)
-		(pin "3"
-		)
-		(pin "4"
-		)
-		(instances
-			(project "battery-node"
-				(path "/0531bb65-44fe-462a-8fbf-92fb22c9abe0/2e6fa66d-cf61-4130-94fd-f989bd2a39c4/14facb8c-7913-48f0-8c95-94965f8c72e2"
-					(reference "CN3")
-					(unit 1)
-				)
-				(path "/0531bb65-44fe-462a-8fbf-92fb22c9abe0/2e6fa66d-cf61-4130-94fd-f989bd2a39c4/524a3c24-e1d4-440c-a5de-5fa78cca8f92"
-					(reference "CN2")
-					(unit 1)
-				)
-				(path "/0531bb65-44fe-462a-8fbf-92fb22c9abe0/2e6fa66d-cf61-4130-94fd-f989bd2a39c4/5ed4f55b-1488-4427-9d20-f9a6669b64e7"
-					(reference "CN1")
-					(unit 1)
-				)
-				(path "/0531bb65-44fe-462a-8fbf-92fb22c9abe0/2e6fa66d-cf61-4130-94fd-f989bd2a39c4/a9e3e829-22d3-464f-b954-379e2fb6907f"
-					(reference "CN4")
-					(unit 1)
-				)
-			)
-		)
-	)
-	(symbol
 		(lib_id "PCM_JLCPCB-Capacitors:0402,470pF")
 		(at 135.89 93.98 0)
@@
 					(unit 1)
 				)
+			)
+		)
+	)
+	(symbol
+		(lib_id "JLCImport:SM02B-NSHSS-TB_LF_SN")
+		(at 116.84 90.17 180)
+		(unit 1)
+		(body_style 1)
+		(exclude_from_sim no)
+		(in_bom yes)
+		(on_board yes)
+		(in_pos_files yes)
+		(dnp no)
+		(fields_autoplaced yes)
+		(property "Reference" "P1"
+			(at 108.4581 90.2278 0)
+			(show_name no)
+			(do_not_autoplace no)
+			(effects
+				(font
+					(size 1.27 1.27)
+				)
+				(justify left)
+			)
+		)
+		(property "Value" "SM02B-NSHSS-TB_LF_SN"
+			(at 108.4581 92.6521 0)
+			(show_name no)
+			(do_not_autoplace no)
+			(effects
+				(font
+					(size 1.27 1.27)
+				)
+				(justify left)
+			)
+		)
+		(property "Footprint" "JLCImport:SM02B-NSHSS-TB_LF_SN"
+			(at 116.84 90.17 0)
+			(hide yes)
+			(show_name no)
+			(do_not_autoplace no)
+			(effects
+				(font
+					(size 1.27 1.27)
+				)
+			)
+		)
+		(property "Datasheet" "https://www.lcsc.com/datasheet/lcsc_datasheet_1811031616_JST-SM02B-NSHSS-TB-LF-SN_C265415.pdf"
+			(at 116.84 90.17 0)
+			(hide yes)
+			(show_name no)
+			(do_not_autoplace no)
+			(effects
+				(font
+					(size 1.27 1.27)
+				)
+			)
+		)
+		(property "Description" "-25℃~+85℃ 1 1A 1x3P (Missing 1P) 2P (3P Missing 1P) 2mm 3 4.4mm 50V 5mm 6.8mm Copper alloy Missing pin、Auxiliary Solder Pin NSH PA Surface Mount, Right Angle Tin UL94V-0 White SMD,P=2mm,卧贴 Wire To Board Connector ROHS"
+			(at 116.84 90.17 0)
+			(hide yes)
+			(show_name no)
+			(do_not_autoplace no)
+			(effects
+				(font
+					(size 1.27 1.27)
+				)
+			)
+		)
+		(property "LCSC" "C265415"
+			(at 116.84 90.17 0)
+			(hide yes)
+			(show_name no)
+			(do_not_autoplace no)
+			(effects
+				(font
+					(size 1.27 1.27)
+				)
+			)
+		)
+		(property "Manufacturer" "JST"
+			(at 116.84 90.17 0)
+			(hide yes)
+			(show_name no)
+			(do_not_autoplace no)
+			(effects
+				(font
+					(size 1.27 1.27)
+				)
+			)
+		)
+		(property "Manufacturer Part" "SM02B-NSHSS-TB(LF)(SN)"
+			(at 116.84 90.17 0)
+			(hide yes)
+			(show_name no)
+			(do_not_autoplace no)
+			(effects
+				(font
+					(size 1.27 1.27)
+				)
+			)
+		)
+		(pin "1"
+		)
+		(pin "3"
+		)
+		(pin "2"
+		)
+		(pin "4"
+		)
+		(instances
+			(project "battery-node"
+				(path "/0531bb65-44fe-462a-8fbf-92fb22c9abe0/2e6fa66d-cf61-4130-94fd-f989bd2a39c4/14facb8c-7913-48f0-8c95-94965f8c72e2"
+					(reference "P3")
+					(unit 1)
+				)
+				(path "/0531bb65-44fe-462a-8fbf-92fb22c9abe0/2e6fa66d-cf61-4130-94fd-f989bd2a39c4/524a3c24-e1d4-440c-a5de-5fa78cca8f92"
+					(reference "P2")
+					(unit 1)
+				)
+				(path "/0531bb65-44fe-462a-8fbf-92fb22c9abe0/2e6fa66d-cf61-4130-94fd-f989bd2a39c4/5ed4f55b-1488-4427-9d20-f9a6669b64e7"
+					(reference "P1")
+					(unit 1)
+				)
+				(path "/0531bb65-44fe-462a-8fbf-92fb22c9abe0/2e6fa66d-cf61-4130-94fd-f989bd2a39c4/a9e3e829-22d3-464f-b954-379e2fb6907f"
+					(reference "P4")
+					(unit 1)
+				)

Commit message: diagonal
Parts:
- removed P1: SM02B-NSHSS-TB_LF_SN, JLCImport:SM02B-NSHSS-TB_LF_SN, symbol JLCImport:SM02B-NSHSS-TB_LF_SN
- added C56: 470pF, PCM_JLCPCB:C_0402, symbol PCM_JLCPCB-Capacitors:0402,470pF
- added CN2: S4B-ZR-SM4A-TF_LF_SN, JLCImport:JST_ZH_S4B-ZR-SM4A-TF_1x04-1MP_P1.50mm_Horizontal, symbol JLCImport:S4B-ZR-SM4A-TF_LF_SN
Connections:
- net GND: now also C56.2, CN2.1, CN2.3, CN2.5, CN2.6
- net THERMISTOR_CHANNEL renamed THERMISTOR_CHANNEL_A
- net THERMISTOR_CHANNEL_A: now also CN2.4
- new net THERMISTOR_CHANNEL_B: C56.1, CN2.2
Other:
- note removed: "use smaller connector"

Commit message: kicad 10.0.1 before update to .2
Connections:
- net GND: now also CN2.MP (5); no longer CN2.5, CN2.6
Changed lines of the file:
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@@
 		(pin "3"
 		)
-		(pin "6"
+		(pin "MP"
 		)
 		(pin "4"
 		)
-		(pin "5"
+		(pin "MP"
 		)
 		(instances

Commit message: done with layout, need to address some DRC
Parts:
- renumbered CN2 to CN4
Changed lines of the file:
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@@
 		(dnp no)
 		(fields_autoplaced yes)
-		(property "Reference" "CN2"
+		(property "Reference" "CN4"
 			(at 98.298 92.7678 0)
 			(show_name no)
@@
 			(project "battery-node"
 				(path "/0531bb65-44fe-462a-8fbf-92fb22c9abe0/2e6fa66d-cf61-4130-94fd-f989bd2a39c4/5ed4f55b-1488-4427-9d20-f9a6669b64e7"
-					(reference "CN2")
+					(reference "CN4")
 					(unit 1)
 				)
